File: projects/OpenSDA Update/obc.sch (EAGLE design)
At the start: 230 parts, among them IC1 IS42S16160J-6BLI, IC2 S26KS512SDPBHI020, IC3 74LVC2T45GS,115, IC4 74LVCH1T45GS,132, IC5 MP2144GJ-Z, IC7 74LVCH1T45GS,132, IC8 74LVCH1T45GS,132, J2 DX4R205JJAR1800, Q1 FA-128, Q3 FC-12M, U1 MIMXRT1052DVL6A, U4 MK20DX128VFM5, U5 NLX2G14CMUTCG, U6 NTSX2102GU8H, U8 NX5P3090UKZ, U9 TC1270ASVRCTR

Commit message: updated schematic and layout of the OBC (with BOM)
Parts:
- removed C83, C84: 10uF, rcl:C-EUC0402K
- removed C85, C88, C91, C92, C95, C96, C97: 0.1uF, rcl:C-EUC0402K
- removed C86: 0.22uF, rcl:C-EUC0402K
- removed C87: 22uF, rcl:C-EUC0402K
- removed C89, C90, C93: 1000pF, rcl:C-EUC0402K
- removed C94: 1.0uF, rcl:C-EUC0402K
- removed D2: (no value), diode:SCHOTTKY-DIODESMC
- removed D6, D7: BAT60J, diode:BAT60J
- removed IC5: MP2144GJ-Z, MP2144GJ-Z:MP2144GJ-Z
- removed L6, L7: 330 Ohm, inductors:B82132
- removed L9: 1uH, rcl:L-EU0204V
- removed R101, R105, R115, R132, R133, R8: 0 Ohm, rcl:R-EU_R0402
- removed R102: 10k Ohm, rcl:R-EU_R0402
- removed R103: 180k Ohm, rcl:R-EU_R0402
- removed R104: 40.2k Ohm, rcl:R-EU_R0402
- removed R112: 100 Ohm, rcl:R-EU_R0402
- removed R113: 1M Ohm, rcl:R-EU_R0402
- removed TP16: TPTP06R, testpad:TPTP06R
- added C38, C50: 0.1uF, rcl:C-EUC0402K
- added C49: 4.7uF, rcl:C-EUC0402K
- added FB1, FB2: MPZ1608S331A, MPZ1608S331A:MPZ1608S331A
- added J1, J3, J4, J5: 504050-0791, 504050-0791:504050-0791
- added J6: 504050-0891, 504050-0891:504050-0891
- added J7: FH28-10S-0.5SH_05_, FH28-10S-0.5SH_05_:FH28-10S-0.5SH_05_
- added J8, J9: ESQ-126-39-G-D, ESQ-126-39-G-D:ESQ-126-39-G-D
- added TP2, TP3: TPTP06R, testpad:TPTP06R
- added U10, U11, U12: HONEYWELL_HMC5983-TRHONEYWELL_HMC5983-TR_0_0, Honeywell - HMC5983-TR:HONEYWELL_HMC5983-TRHONEYWELL_HMC5983-TR_0_0
- added U2: MCP1702T-1802E/CB, MCP1702T1802ECB:MCP1702T-1802E/CB
- added U3, U7: NXP_FXAS21002CQR1NXP_FXAS21002CQR1_0_0, NXP - FXAS21002CQR1:NXP_FXAS21002CQR1NXP_FXAS21002CQR1_0_0
- C32: value 0.1uF -> 10uF
- L2: value 4.7uH -> 4.7 uH; device rcl:L-EUL4035M -> inductors:BLM15HB121SN1
- R4: value 1K Ohm -> 0 Ohm
- U9: value TC1270ASVRCTR -> NXP_FXAS21002CQR1NXP_FXAS21002CQR1_0_0; device TC1270ASVRCTR:TC1270ASVRCTR -> NXP - FXAS21002CQR1:NXP_FXAS21002CQR1NXP_FXAS21002CQR1_0_0
Connections:
- removed net 5V_SYS: R101.1, R114.2
- removed net MCU_DCDC_IN_3V3: C95.1, R115.2, R7.2
- removed net N$61: C83.2, C84.2, C85.2, IC5.VIN, R101.2
- removed net N$62: C86.1, IC5.EN, R102.2, U9.!RESET
- removed net N$63: C89.1, C90.1, IC5.PG, TP16.TP
- removed net N$64: IC5.SW, L9.2
- removed net N$67: IC5.FB, R103.1, R104.2
- removed net N$68: D6.A, D7.A, U9.!MR
- removed net N$71: C93.1, D6.C, R112.2
- removed net N$74: C94.2, D7.C, R113.2
- removed net POR_BUTTON: R112.1
- removed net VDDA_ADC_3V3: C14.1, C15.1, C97.1, R1.1, R1.2, R133.2, U1.VDDA_ADC_3P3
- removed net VDD_COIN_3V: D2.A, R4.2
- removed net VDD_HIGH_IN_3V3: C18.1, C19.1, C96.1, R132.2, U1.VDD_HIGH_IN
- removed net VDD_SNVS_3V3: C91.1, D1.A, R105.2
- removed net VDD_SVNS_3V3: C92.1, U9.VCC
- new net LDO_1V8: C49.1, C50.1, R4.1, TP3.TP, U2.VOUT
- new net N$40: C32.1, C38.1, R1.1, U2.VIN
- net DCDC_3V3: now also C14.1, C15.1, C18.1, C19.1, D1.A, R1.2, R114.2, R7.2, U1.VDDA_ADC_3P3, U1.VDD_HIGH_IN; no longer C87.1, C88.1, IC5.OUT, L9.1, R103.2, R105.1, R115.1, R132.1, R133.1, R8.1
- net FLASH_VCC: now also R4.2; no longer C32.1, R8.2
- net GND: now also C38.2, C49.2, C50.2, FB2.1, U2.GND; no longer C83.1, C84.1, C85.1, C86.2, C87.2, C88.2, C89.2, C90.2, C91.2, C92.2, C93.2, C95.2, C96.2, C97.2, IC5.AGND, IC5.PGND, L7.1, R104.1, R113.1, U9.GND
- net N$5: no longer D2.C, R4.1
- net ONOFF: now also TP2.TP
- net P5V0_SDA_USB_CONN_VBUS: now also FB1.1; no longer L6.1
- net P5V_SDA: now also FB1.2; no longer L6.2
- net PMIC_ON_REQ: no longer R102.1
- net SDA_USBSHIELD: now also FB2.2; no longer L7.2
- net WDOG_B: no longer C94.1
Other:
- note removed: "missing JTAG connector"
